Commit message: merging the ur5 to husky

File: src/husky_isaac_sim/urdf/husky_ur5.urdf (robot description, URDF)
Before this commit: robot husky_ur5, 37 links, 36 joints
Links:
- link husky_base_link: geometry collision box size=0.7899200000000001 0.5709 0.10375; collision box size=0.9874 0.5709 0.12375
- link husky_front_bumper_link: geometry visual mesh filename=file:///home/dada/raicam_ws/summit_arm_sim/src/husky_descri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
- link husky_front_left_wheel: geometry collision cylinder length=0.1143 radius=0.1651; visual mesh filename=file:///home/dada/raicam_ws/summit_arm_sim/src/husky_descri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
- link husky_front_right_wheel: geometry collision cylinder length=0.1143 radius=0.1651; visual mesh filename=file:///home/dada/raicam_ws/summit_arm_sim/src/husky_descri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
- link husky_rear_bumper_link: geometry visual mesh filename=file:///home/dada/raicam_ws/summit_arm_sim/src/husky_descri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
- link husky_rear_left_wheel: geometry collision cylinder length=0.1143 radius=0.1651; visual mesh filename=file:///home/dada/raicam_ws/summit_arm_sim/src/husky_descri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
- link husky_rear_right_wheel: geometry collision cylinder length=0.1143 radius=0.1651; visual mesh filename=file:///home/dada/raicam_ws/summit_arm_sim/src/husky_descri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
- link husky_sensor_arch_mount_link: geometry collision mesh filename=file:///home/dada/raicam_ws/summit_arm_sim/src/husky_descri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; visual mesh filename=file:///home/dada/raicam_ws/summit_arm_sim/src/husky_descri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
- link husky_top_chassis_link: geometry visual mesh filename=file:///home/dada/raicam_ws/summit_arm_sim/src/husky_descri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
- link husky_top_plate_link: geometry collision mesh filename=file:///home/dada/raicam_ws/summit_arm_sim/src/husky_descri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; visual mesh filename=file:///home/dada/raicam_ws/summit_arm_sim/src/husky_descri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
- link husky_user_rail_link: geometry visual mesh filename=file:///home/dada/raicam_ws/summit_arm_sim/src/husky_descri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

File: src/ur5_isaac_simulation/urdfur5_robotiq.urdf (robot description, URDF)
Before this commit: robot husky_ur5, 37 links, 36 joints
Links:
- link husky_base_link: geometry collision box size=0.7899200000000001 0.5709 0.10375; collision box size=0.9874 0.5709 0.12375
- link husky_front_bumper_link: geometry visual mesh filename=file:///home/dada/raicam_ws/summit_arm_sim/src/husky_descri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
- link husky_front_left_wheel: geometry collision cylinder length=0.1143 radius=0.1651; visual mesh filename=file:///home/dada/raicam_ws/summit_arm_sim/src/husky_descri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
- link husky_front_right_wheel: geometry collision cylinder length=0.1143 radius=0.1651; visual mesh filename=file:///home/dada/raicam_ws/summit_arm_sim/src/husky_descri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
- link husky_rear_bumper_link: geometry visual mesh filename=file:///home/dada/raicam_ws/summit_arm_sim/src/husky_descri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
- link husky_rear_left_wheel: geometry collision cylinder length=0.1143 radius=0.1651; visual mesh filename=file:///home/dada/raicam_ws/summit_arm_sim/src/husky_descri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
- link husky_rear_right_wheel: geometry collision cylinder length=0.1143 radius=0.1651; visual mesh filename=file:///home/dada/raicam_ws/summit_arm_sim/src/husky_descri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
- link husky_sensor_arch_mount_link: geometry collision mesh filename=file:///home/dada/raicam_ws/summit_arm_sim/src/husky_descri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; visual mesh filename=file:///home/dada/raicam_ws/summit_arm_sim/src/husky_descri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
- link husky_top_chassis_link: geometry visual mesh filename=file:///home/dada/raicam_ws/summit_arm_sim/src/husky_descri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
- link husky_top_plate_link: geometry collision mesh filename=file:///home/dada/raicam_ws/summit_arm_sim/src/husky_descri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; visual mesh filename=file:///home/dada/raicam_ws/summit_arm_sim/src/husky_descri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
- link husky_user_rail_link: geometry visual mesh filename=file:///home/dada/raicam_ws/summit_arm_sim/src/husky_descri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
- link left_inner_finger: geometry collision mesh filename=/home/dada/raicam_ws/summit_arm_sim/src/ur5_isaac_simulatio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; visual mesh filename=/home/dada/raicam_ws/summit_arm_sim/src/ur5_isaac_simulatio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
- link left_inner_knuckle: geometry collision mesh filename=/home/dada/raicam_ws/summit_arm_sim/src/ur5_isaac_simulatio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; visual mesh filename=/home/dada/raicam_ws/summit_arm_sim/src/ur5_isaac_simulatio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
- link left_outer_finger: geometry collision mesh filename=/home/dada/raicam_ws/summit_arm_sim/src/ur5_isaac_simulatio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; visual mesh filename=/home/dada/raicam_ws/summit_arm_sim/src/ur5_isaac_simulatio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
- link left_outer_knuckle: geometry collision mesh filename=/home/dada/raicam_ws/summit_arm_sim/src/ur5_isaac_simulatio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; visual mesh filename=/home/dada/raicam_ws/summit_arm_sim/src/ur5_isaac_simulatio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
- link right_inner_finger: geometry collision mesh filename=/home/dada/raicam_ws/summit_arm_sim/src/ur5_isaac_simulatio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; visual mesh filename=/home/dada/raicam_ws/summit_arm_sim/src/ur5_isaac_simulatio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
- link right_inner_knuckle: geometry collision mesh filename=/home/dada/raicam_ws/summit_arm_sim/src/ur5_isaac_simulatio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; visual mesh filename=/home/dada/raicam_ws/summit_arm_sim/src/ur5_isaac_simulatio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
- link right_outer_finger: geometry collision mesh filename=/home/dada/raicam_ws/summit_arm_sim/src/ur5_isaac_simulatio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; visual mesh filename=/home/dada/raicam_ws/summit_arm_sim/src/ur5_isaac_simulatio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
- link right_outer_knuckle: geometry collision mesh filename=/home/dada/raicam_ws/summit_arm_sim/src/ur5_isaac_simulatio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; visual mesh filename=/home/dada/raicam_ws/summit_arm_sim/src/ur5_isaac_simulatio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
- link robotiq_arg2f_base_link: geometry collision mesh filename=/home/dada/raicam_ws/summit_arm_sim/src/ur5_isaac_simulatio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; visual mesh filename=/home/dada/raicam_ws/summit_arm_sim/src/ur5_isaac_simulatio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
- link ur5_base_link_inertia: geometry collision mesh filename=/home/dada/raicam_ws/summit_arm_sim/src/ur5_isaac_simulatio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; visual mesh filename=/home/dada/raicam_ws/summit_arm_sim/src/ur5_isaac_simulatio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
- link ur5_forearm_link: geometry collision mesh filename=/home/dada/raicam_ws/summit_arm_sim/src/ur5_isaac_simulatio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; visual mesh filename=/home/dada/raicam_ws/summit_arm_sim/src/ur5_isaac_simulatio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
- link ur5_shoulder_link: geometry collision mesh filename=/home/dada/raicam_ws/summit_arm_sim/src/ur5_isaac_simulatio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; visual mesh filename=/home/dada/raicam_ws/summit_arm_sim/src/ur5_isaac_simulatio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
- link ur5_upper_arm_link: geometry collision mesh filename=/home/dada/raicam_ws/summit_arm_sim/src/ur5_isaac_simulatio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; visual mesh filename=/home/dada/raicam_ws/summit_arm_sim/src/ur5_isaac_simulatio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
- link ur5_wrist_1_link: geometry collision mesh filename=/home/dada/raicam_ws/summit_arm_sim/src/ur5_isaac_simulatio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; visual mesh filename=/home/dada/raicam_ws/summit_arm_sim/src/ur5_isaac_simulatio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
- link ur5_wrist_2_link: geometry collision mesh filename=/home/dada/raicam_ws/summit_arm_sim/src/ur5_isaac_simulatio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; visual mesh filename=/home/dada/raicam_ws/summit_arm_sim/src/ur5_isaac_simulatio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
- link ur5_wrist_3_link: geometry collision mesh filename=/home/dada/raicam_ws/summit_arm_sim/src/ur5_isaac_simulatio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; visual mesh filename=/home/dada/raicam_ws/summit_arm_sim/src/ur5_isaac_simulatio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
